File: kicad/picopet/picopet.kicad_pcb (KiCad board)
At the start: 2 copper layers, 56 parts, among them J1 USB_C_Receptacle_USB2.0_14P, J2 PH1.25mm 2P, J3 PH1.25mm 2P, J4 CR1220 Holder, J5 ST7735 LCD, Q1 SS8050, SW1 PWR, SW2 BOOTSEL, SW3 Btn0, SW4 Btn1, SW5 Btn2, SW6 Btn3, U1 RP2040, U2 MCP73831-2-OT, U3 S-T111B33MC-OGSTFU, U4 DS3231MZ, U6 AT24CS32-SSHM, U7 W25Q32JVSSIQ, Y1 X322512MSB4SI

Commit message: Tons of changes regarding batteries...
Parts:
- removed C17, C18: 1u, Capacitor_SMD:C_0805_2012Metric
- removed C19: 4.7u, Capacitor_SMD:C_0805_2012Metric
- removed J2: PH1.25mm 2P, Connector_JST:JST_GH_SM02B-GHS-TB_1x02-1MP_P1.25mm_Horizontal
- removed R12: 5k1, Resistor_SMD:R_0201_0603Metric
- removed R8, R9: 100k, Resistor_SMD:R_0402_1005Metric
- removed U2: MCP73831-2-OT, Package_TO_SOT_SMD:SOT-23-5
- removed U3: S-T111B33MC-OGSTFU, Package_TO_SOT_SMD:SOT-23-5
- BZ1: footprint Buzzer_Beeper:MagneticBuzzer_Kobitone_254-EMB84Q-RO -> Buzzer_Beeper:Buzzer_CUI_CPT-9019S-SMT
- SW1: footprint Button_Switch_SMD:SW_SPDT_CK_JS102011SAQN -> Button_Switch_THT:SW_Slide_SPDT_Angled_CK_OS102011MA1Q
- moved SW1 2.65 mm to (16.0, 129.5)
- moved BZ1 1.83 mm to (40.0, 128.5), turned to 180 degrees
Routing:
- net VSENSE: track 17.6 -> 0.00 mm
- net VBAT: track 11.5 -> 0.00 mm
- net GND: track 31.6 -> 21.5 mm
- net +3V3: track 78.2 -> 76.2 mm
- net USBC_VDD: track 10.6 -> 8.73 mm
- net Net-(U2-PROG): track 1.20 -> 0.00 mm
- net GPIO26: track 0.88 -> 0.00 mm
