File: kicad/picopet/picopet.kicad_sch (KiCad schematic)
At the start: 56 parts, among them J1 USB_C_Receptacle_USB2.0_14P, J2 PH1.25mm 2P, J3 PH1.25mm 2P, J4 CR1220 Holder, J5 ST7735 LCD, Q1 SS8050, SW1 PWR, SW2 BOOTSEL, SW3 Btn0, SW4 Btn1, SW5 Btn2, SW6 Btn3, U1 RP2040, U2 MCP73831-2-OT, U3 S-T111B33MC-OGSTFU, U4 DS3231MZ, U6 AT24CS32-SSHM, U7 W25Q32JVSSIQ, Y1 X322512MSB4SI

Commit message: Tons of changes regarding batteries...
Parts:
- BZ1: footprint Buzzer_Beeper:MagneticBuzzer_Kobitone_254-EMB84Q-RO -> Buzzer_Beeper:Buzzer_CUI_CPT-9019S-SMT
